File: EC200_INTERFACE.kicad_sch (KiCad schematic)
At the start: 29 parts, among them J3 U.FL-R-SMT_01_, J4 MSIM-12-A, SW1 SW_Push, SW2 SW_Push, U6 TXS0102DCT, U7 EC200UCNAB-N05-SNNSA, U8 ST4SI2M0020TPIFW, U9 TS3A27518EPW

Commit message: Update buck 5-3.8V and change mosfet
Parts:
- C36: renamed from C34; footprint Capacitor_Tantalum_SMD:CP_EIA-7343-31_Kemet-D -> Capacitor_Tantalum_SMD:CP_EIA-3528-12_Kemet-T_HandSolder
- C38: renamed from C36; footprint Capacitor_Tantalum_SMD:CP_EIA-7343-31_Kemet-D -> Capacitor_Tantalum_SMD:CP_EIA-3528-12_Kemet-T_HandSolder
- renumbered C30 to C32, C31 to C33, C32 to C34, C33 to C35, C35 to C37, C37 to C39, C38 to C40, C39 to C41, C40 to C42, C41 to C43, C42 to C44, C43 to C45, C44 to C46, C45 to C47, C46 to C48, D7 to D8, D8 to D9, R30 to R32, R31 to R33

Commit message: Change POWER_CHARGE
Parts:
- renumbered C32 to C19, C33 to C20, C34 to C21, C35 to C22, C36 to C23, C37 to C24, C38 to C25, C39 to C26, C40 to C27, C41 to C28, C42 to C29, C43 to C30, C44 to C31, C45 to C32, C46 to C33, C47 to C34, C48 to C35, R32 to R17, R33 to R18
