File: MCU.kicad_sch (KiCad schematic)
At the start: 51 parts, among them J5 KH-TYPE-C-16P, J6 Conn_01x04_Pin, SW3 SW_Push, SW4 SW_Push, SW5 SW_Push, U10 W25Q32JVSS, U11 STM32H743VITx, U12 MAX809TEUR_T, U13 AP2112K-3.3, Y1 25MHz_Crystal_GND24 _8Z250000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, Y2 Crystal_32.768K

Commit message: Update buck 5-3.8V and change mosfet
Parts:
- renumbered C47 to C49, C48 to C50, C49 to C51, C50 to C52, C51 to C53, C52 to C54, C53 to C55, C54 to C56, C55 to C57, C56 to C58, C57 to C59, C58 to C60, C59 to C61, C60 to C62, C61 to C63, C62 to C64, C63 to C65, C64 to C66, C65 to C67, C66 to C68, C67 to C69, C68 to C70, D9 to D10, D10 to D11, D11 to D12, D12 to D13, D13 to D14, D14 to D15, R32 to R34, R33 to R35, R34 to R36, R35 to R37, R36 to R38, R37 to R39, R38 to R40, R39 to R41, R40 to R42, R41 to R43, R42 to R44

Commit message: Change POWER_CHARGE
Parts:
- renumbered C49 to C36, C50 to C37, C51 to C38, C52 to C39, C53 to C40, C54 to C41, C55 to C42, C56 to C43, C57 to C44, C58 to C45, C59 to C46, C60 to C47, C61 to C48, C62 to C49, C63 to C50, C64 to C51, C65 to C52, C66 to C53, C67 to C54, C68 to C55, C69 to C56, C70 to C57, R34 to R19, R35 to R20, R36 to R21, R37 to R22, R38 to R23, R39 to R24, R40 to R25, R41 to R26, R42 to R27, R43 to R28, R44 to R29
