File: POWER_MANAGEMENT.kicad_sch (KiCad schematic)
At the start: 18 parts, among them U4 TPS62130A, U5 TPS5430DDA

Commit message: Update buck 5-3.8V and change mosfet
Parts:
- removed C22: 3.3nF, Capacitor_SMD:C_0805_2012Metric_Pad1.18x1.45mm_HandSolder, symbol Device:C
- removed C23, C28: 470uF, Capacitor_Tantalum_SMD:CP_EIA-7343-31_Kemet-D, symbol Device:C_Polarized
- removed C25: 10uF, Capacitor_SMD:C_0805_2012Metric_Pad1.18x1.45mm_HandSolder, symbol Device:C
- removed L2: 1uH, Inductor_SMD:L_Abracon_ASPI-0425, symbol Device:L
- removed U4: TPS62130A, Package_DFN_QFN:VQFN-16-1EP_3x3mm_P0.5mm_EP1.68x1.68mm_ThermalVias, symbol Regulator_Switching:TPS62130A
- added C22, C30: 470uF, Capacitor_Tantalum_SMD:CP_EIA-7343-31_Kemet-D, symbol Device:C_Polarized
- added C23, C31: 0.1uF, Capacitor_SMD:C_0805_2012Metric_Pad1.18x1.45mm_HandSolder, symbol Device:C
- added C26: 22uF, Capacitor_SMD:C_0805_2012Metric_Pad1.18x1.45mm_HandSolder, symbol Device:C
- added C28: 10pF, Capacitor_SMD:C_0805_2012Metric_Pad1.18x1.45mm_HandSolder, symbol Device:C
- added D7: B340A, Diode_SMD:D_SMC, symbol Diode:B340
- added L3: 2.5uH, Inductor_SMD:L_Abracon_ASPI-0425, symbol Device:L_Iron
- added R30: 18.7k, Resistor_SMD:R_0805_2012Metric, symbol Device:R
- added R31: 4.99k, Resistor_SMD:R_0805_2012Metric, symbol Device:R
- added U5: TPS54332DDA, footprintf:VREG_LM5017MR_NOPB, symbol symbol:TPS54332DDA
- C24: value 0.1uF -> 0.015uF
- C27: value 100nF -> 180pF
- C29: footprint Capacitor_Tantalum_SMD:CP_EIA-3216-10_Kemet-I_HandSolder -> Capacitor_Tantalum_SMD:CP_EIA-7343-31_Kemet-D
- R26: value 374K -> 1M
- R27: value 100K -> 75k
- renumbered C26 to C25, L3 to L2, U5 to U4
Connections:
- net GND: now also R26.2, C22.2, C23.1, C26.1, C28.1, C30.2, C31.1, D7.2 (A), R31.2, U5.7 (GND), U5.9 (EP); no longer C27.1
- net V_OUT-3.8V: now also C30.1, C31.2, L3.2, R30.1; no longer C27.2, R26.1
- net V_OUT-5V: now also C22.1, C23.2, U5.2 (VIN), U5.3 (EN); no longer C24.2
- net at R27.1: now also C27.1; no longer R26.2
- new net: C27.2, C28.2, U5.6 (COMP)
- new net: C24.2, R26.1, U5.4 (SS)
- new net: C26.2, D7.1 (K), L3.1, U5.1 (BOOT), U5.8 (PH)
- new net: R30.2, R31.1, U5.5 (VSENSE)
- no-connect marks 1 -> 0

Commit message: Change POWER_CHARGE
Parts:
- renumbered C23 to C10, C24 to C11, C25 to C12, C26 to C13, C27 to C14, C28 to C15, C29 to C16, C30 to C17, C31 to C18, C21 to C8, C22 to C9, R26 to R11, R27 to R12, R28 to R13, R29 to R14, R30 to R15, R31 to R16
Other:
- moved on the sheet: C13
