File: RS_INTERFACE.kicad_sch (KiCad schematic)
At the start: 55 parts, among them IC1 ADM3251EARWZ-REEL, IC2 ADM3251EARWZ-REEL, J10 Screw_Terminal_01x03, J11 Screw_Terminal_01x03, J7 Screw_Terminal_01x05, J8 Screw_Terminal_01x05, J9 Screw_Terminal_01x05, U14 ISO1211, U15 ISO1211, U16 ISO1211, U17 ISO1211, U18 ADM2587E, U19 ADM2587E

Commit message: Update buck 5-3.8V and change mosfet
Parts:
- renumbered C98 to C100, C99 to C101, C100 to C102, C69 to C71, C70 to C72, C71 to C73, C72 to C74, C73 to C75, C74 to C76, C75 to C77, C76 to C78, C77 to C79, C78 to C80, C79 to C81, C80 to C82, C81 to C83, C82 to C84, C83 to C85, C84 to C86, C85 to C87, C86 to C88, C87 to C89, C88 to C90, C89 to C91, C90 to C92, C91 to C93, C92 to C94, C93 to C95, C94 to C96, C95 to C97, C96 to C98, C97 to C99, R43 to R45, R44 to R46, R45 to R47, R46 to R48, R47 to R49, R48 to R50, R49 to R51, R50 to R52

Commit message: Change POWER_CHARGE
Parts:
- renumbered C71 to C58, C72 to C59, C73 to C60, C74 to C61, C75 to C62, C76 to C63, C77 to C64, C78 to C65, C79 to C66, C80 to C67, C81 to C68, C82 to C69, C83 to C70, C84 to C71, C85 to C72, C86 to C73, C87 to C74, C88 to C75, C89 to C76, C90 to C77, C91 to C78, C92 to C79, C93 to C80, C94 to C81, C95 to C82, C96 to C83, C97 to C84, C98 to C85, C99 to C86, C100 to C87, C101 to C88, C102 to C89, IC1 to IC2, IC2 to IC3, R45 to R30, R46 to R31, R47 to R32, R48 to R33, R49 to R34, R50 to R35, R51 to R36, R52 to R37
Connections:
- net GND2: no longer C70.2, C72.2, C74.2, C76.2, C88.2
- net GND_RS232: now also C88.2
- net GND_RS485: now also C70.2, C72.2, C74.2, C76.2
