File: loc.kicad_pcb (KiCad board)
At the start: 2 copper layers, 100 x 100 mm, 214 parts, among them IC1 ADM3251EARWZ-REEL, IC2 ADM3251EARWZ-REEL, J1 Screw_Terminal_01x02, J10 Screw_Terminal_01x03, J11 Screw_Terminal_01x03, J2 Screw_Terminal_01x03, J3 U.FL-R-SMT_01_, J4 MSIM-12-A, J5 KH-TYPE-C-16P, J6 Conn_01x04_Pin, J7 Screw_Terminal_01x05, J8 Screw_Terminal_01x05, J9 Screw_Terminal_01x05, Q1 Si7617DN, Q2 Si7617DN, Q3 SiS412DN, Q4 SiS412DN, Q5 Si7617DN, SW1 SW_Push, SW2 SW_Push, SW3 SW_Push, SW4 SW_Push, SW5 SW_Push, U1 STN8205A, U10 W25Q32JVSS, U11 STM32H743VITx, U12 MAX809TEUR_T, U13 AP2112K-3.3, U14 ISO1211, U15 ISO1211, U16 ISO1211, U17 ISO1211, U18 ADM2587E, U19 ADM2587E, U2 HY22120-CB, U3 BQ24610, U4 TPS62130A, U5 TPS5430DDA, U6 TXS0102DCT, U7 EC200UCNAB-N05-SNNSA, U8 ST4SI2M0020TPIFW, U9 TS3A27518EPW, Y1 25MHz_Crystal_GND24 _8Z250000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, Y2 Crystal_32.768K

Commit message: Update buck 5-3.8V and change mosfet
Parts:
- removed the C25 at (217.2, 41.2)
- removed the L2 at (168.3, 158.5)
- removed the U4 at (228.5, 42.8)
- added C26: 22uF, Capacitor_SMD:C_0805_2012Metric_Pad1.18x1.45mm_HandSolder, F.Cu at (69.5, 111.1)
- added C30: 470uF, Capacitor_Tantalum_SMD:CP_EIA-7343-31_Kemet-D, F.Cu at (76.8, 109.3)
- added C31: 0.1uF, Capacitor_SMD:C_0805_2012Metric_Pad1.18x1.45mm_HandSolder, F.Cu at (69.5, 108.1)
- added D7: B340A, Diode_SMD:D_SMC, F.Cu at (77.3, 116.1)
- added L3: 2.5uH, Inductor_SMD:L_Abracon_ASPI-0425, F.Cu at (74.9, 122.8)
- added R30: 18.7k, Resistor_SMD:R_0805_2012Metric, F.Cu at (85.0, 119.6)
- added R31: 4.99k, Resistor_SMD:R_0805_2012Metric, F.Cu at (85.0, 122.6)
- added U5: TPS54332DDA, footprintf:VREG_LM5017MR_NOPB, F.Cu at (91.3, 103.8)
- C1: footprint Capacitor_Tantalum_SMD:CP_EIA-3216-10_Kemet-I_HandSolder -> Capacitor_Tantalum_SMD:CP_EIA-3528-12_Kemet-T_HandSolder
- C22: value 3.3nF -> 470uF; footprint Capacitor_SMD:C_0805_2012Metric_Pad1.18x1.45mm_HandSolder -> Capacitor_Tantalum_SMD:CP_EIA-7343-31_Kemet-D
- C23: value 470uF -> 0.1uF; footprint Capacitor_Tantalum_SMD:CP_EIA-7343-31_Kemet-D -> Capacitor_SMD:C_0805_2012Metric_Pad1.18x1.45mm_HandSolder
- C24: value 0.1uF -> 0.015uF
- C27: value 100nF -> 180pF
- C28: value 470uF -> 10pF; footprint Capacitor_Tantalum_SMD:CP_EIA-7343-31_Kemet-D -> Capacitor_SMD:C_0805_2012Metric_Pad1.18x1.45mm_HandSolder
- C29: footprint Capacitor_Tantalum_SMD:CP_EIA-3216-10_Kemet-I_HandSolder -> Capacitor_Tantalum_SMD:CP_EIA-7343-31_Kemet-D
- C36: renamed from C34; footprint Capacitor_Tantalum_SMD:CP_EIA-7343-31_Kemet-D -> Capacitor_Tantalum_SMD:CP_EIA-3528-12_Kemet-T_HandSolder
- C38: renamed from C36; footprint Capacitor_Tantalum_SMD:CP_EIA-7343-31_Kemet-D -> Capacitor_Tantalum_SMD:CP_EIA-3528-12_Kemet-T_HandSolder
- Q1, Q2, Q5: value Si7617DN -> AO4407A; footprint Package_SO:Vishay_PowerPAK_1212-8_Single -> footprintf:SOIC127P600X175-8N
- Q3, Q4: value SiS412DN -> FDS6690A; footprint Package_SO:Vishay_PowerPAK_1212-8_Single -> Package_SO:SOIC-8_3.9x4.9mm_P1.27mm
- R26: value 374K -> 1M
- R27: value 100K -> 75k
- moved C42 172.6 mm to (236.9, 46.3)
- moved C43 172.6 mm to (237.1, 76.6)
- moved C47 172.6 mm to (236.8, 70.6)
- moved J4 172.6 mm to (264.4, 58.8)
- moved U8 172.6 mm to (261.5, 77.2)
- moved U9 172.6 mm to (245.6, 53.0)
- moved C40 172.6 mm to (249.4, 74.1)
- moved C41 172.6 mm to (249.4, 65.0)
- moved C44 172.6 mm to (249.4, 68.0)
- moved C45 172.6 mm to (249.4, 80.1)
- moved C46 172.6 mm to (249.4, 71.1)
- moved C48 172.6 mm to (249.4, 77.1)
- moved C24 162.0 mm to (69.5, 105.1)
- moved Q3 161.8 mm to (74.8, 174.3)
- moved C22 155.7 mm to (76.8, 103.5)
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- renumbered C98 to C100, C99 to C101, C100 to C102, C26 to C25, C30 to C32, C31 to C33, C32 to C34, C33 to C35, C35 to C37, C37 to C39, C38 to C40, C39 to C41, C40 to C42, C41 to C43, C42 to C44, C43 to C45, C44 to C46, C45 to C47, C46 to C48, C47 to C49, C48 to C50, C49 to C51, C50 to C52, C51 to C53, C52 to C54, C53 to C55, C54 to C56, C55 to C57, C56 to C58, C57 to C59, C58 to C60, C59 to C61, C60 to C62, C61 to C63, C62 to C64, C63 to C65, C64 to C66, C65 to C67, C66 to C68, C67 to C69, C68 to C70, C69 to C71, C70 to C72, C71 to C73, C72 to C74, C73 to C75, C74 to C76, C75 to C77, C76 to C78, C77 to C79, C78 to C80, C79 to C81, C80 to C82, C81 to C83, C82 to C84, C83 to C85, C84 to C86, C85 to C87, C86 to C88, C87 to C89, C88 to C90, C89 to C91, C90 to C92, C91 to C93, C92 to C94, C93 to C95, C94 to C96, C95 to C97, C96 to C98, C97 to C99, D9 to D10, D10 to D11, D11 to D12, D12 to D13, D13 to D14, D14 to D15, D7 to D8, D8 to D9, L3 to L2, R30 to R32, R31 to R33, R32 to R34, R33 to R35, R34 to R36, R35 to R37, R36 to R38, R37 to R39, R38 to R40, R39 to R41, R40 to R42, R41 to R43, R42 to R44, R43 to R45, R44 to R46, R45 to R47, R46 to R48, R47 to R49, R48 to R50, R49 to R51, R50 to R52, U5 to U4
Connections:
- C13 pad 2: Net-(Q4-D) -> Net-(C13-Pad2)
- C22 pad 1: GND -> /so_do_khoi/RTU_SENSOR_DATA/MCU/V_OUT-5V
- C22 pad 2: Net-(U4-SS/TR) -> GND
- C23 pad 1: /so_do_khoi/RTU_SENSOR_DATA/MCU/V_OUT-5V -> GND
- C23 pad 2: GND -> /so_do_khoi/RTU_SENSOR_DATA/MCU/V_OUT-5V
- C24 pad 2: /so_do_khoi/RTU_SENSOR_DATA/MCU/V_OUT-5V -> Net-(U5-SS)
- C27 pad 1: GND -> Net-(C27-Pad1)
- C27 pad 2: +3V8 -> Net-(U5-COMP)
- C28 pad 1: +3V8 -> GND
- C28 pad 2: GND -> Net-(U5-COMP)
- C5 pad 1: Net-(Q2-D) -> Net-(U3-ACP)
- C7 pad 1: Net-(Q2-D) -> Net-(U3-ACP)
- L1 pad 1: Net-(Q4-D) -> Net-(C13-Pad2)
- Q2 pad 5: Net-(Q2-D) -> Net-(U3-ACP)
- Q4 pad 5: Net-(Q4-D) -> Net-(C13-Pad2)
- R13 pad 1: Net-(Q2-D) -> Net-(U3-ACP)
- R26 pad 1: +3V8 -> Net-(U5-SS)
- R26 pad 2: Net-(U4-FB) -> GND
- R27 pad 1: Net-(U4-FB) -> Net-(C27-Pad1)
- U3 pad 2: Net-(Q2-D) -> Net-(U3-ACP)

Commit message: Change POWER_CHARGE
Parts:
- added C103: 1uF, Capacitor_SMD:C_0805_2012Metric_Pad1.18x1.45mm_HandSolder, F.Cu at (249.5, 122.6)
- added C104: 10uF, Capacitor_SMD:C_0805_2012Metric_Pad1.18x1.45mm_HandSolder, F.Cu at (249.5, 125.6)
- added C105: 0.1uF, Capacitor_SMD:C_0805_2012Metric_Pad1.18x1.45mm_HandSolder, F.Cu at (249.5, 128.6)
- added C106: 10uF, Capacitor_SMD:C_0805_2012Metric_Pad1.18x1.45mm_HandSolder, F.Cu at (249.5, 131.6)
- added D16: B340A, Diode_SMD:D_SMC, F.Cu at (241.7, 111.4)
- added D17: LED, LED_SMD:LED_0805_2012Metric_Pad1.15x1.40mm_HandSolder, F.Cu at (238.6, 124.6)
- added D18: LED, LED_SMD:LED_0805_2012Metric_Pad1.15x1.40mm_HandSolder, F.Cu at (238.6, 127.6)
- added D19: B340A, Diode_SMD:D_SMC, F.Cu at (241.7, 119.2)
- added D21: BAS40, footprintf:SOT23, F.Cu at (243.0, 130.0)
- added IC3: LT3650EMSE-8.4_TRPBF, footprintf:SOP65P490X110-13N, F.Cu at (255.6, 123.9)
- added J12: Screw_Terminal_01x02, TerminalBlock_Phoenix:TerminalBlock_Phoenix_MKDS-3-2-5.08_1x02_P5.08mm_Horizontal, F.Cu at (250.6, 114.5)
- added L4: 6.8uH, Inductor_SMD:L_Abracon_ASPI-0425, F.Cu at (254.9, 129.5)
- added R53: 0.017, Resistor_SMD:R_0805_2012Metric, F.Cu at (234.0, 109.0)
- added R54: 402k, Resistor_SMD:R_0805_2012Metric, F.Cu at (234.0, 112.0)
- added R55: 47k, Resistor_SMD:R_0805_2012Metric, F.Cu at (234.0, 114.9)
- added R56: 10k, Resistor_SMD:R_0805_2012Metric, F.Cu at (234.0, 117.9)
- added R57: 10k, Resistor_SMD:R_0805_2012Metric, F.Cu at (234.0, 120.8)
- added R58: 0.05, Resistor_SMD:R_0805_2012Metric, F.Cu at (234.0, 123.8)
- added U20: LTC4412xS6, Package_TO_SOT_SMD:TSOT-23-6, F.Cu at (243.6, 125.5)
- D2: footprint LED_SMD:LED_1206_3216Metric -> LED_SMD:LED_0805_2012Metric_Pad1.15x1.40mm_HandSolder
- moved R32 6.48 mm to (63.5, 76.6)
- moved D11 5.50 mm to (79.8, 83.3)
- moved C36 1.54 mm to (135.8, 69.8)
- moved R33 0.62 mm to (56.9, 78.1)
- moved J5 0.47 mm to (49.1, 76.4)
- moved IC1 0.16 mm to (124.1, 54.9)
- moved IC2 0.16 mm to (110.0, 55.3)
Connections:
- C101 pad 2: GND2 -> GND_RS232
- C83 pad 2: GND2 -> GND_RS485
- C85 pad 2: GND2 -> GND_RS485
- C87 pad 2: GND2 -> GND_RS485
- C89 pad 2: GND2 -> GND_RS485
Routing:
- net (no net): vias 0 -> 1

Commit message: CHANGE POWWER _CHARGE
Parts:
- removed the C1 at (207.0, 124.3)
- removed the C10 at (76.0, 154.6)
- removed the C11 at (76.0, 151.2)
- removed the C12 at (76.0, 164.6)
- removed the C13 at (81.2, 157.5)
- removed the C14 at (81.2, 160.0)
- removed the C15 at (81.2, 152.5)
- removed the C16 at (81.2, 162.5)
- removed the C17 at (76.0, 157.9)
- removed the C18 at (76.0, 161.3)
- removed the C19 at (76.0, 147.9)
- removed the C20 at (81.2, 165.0)
- removed the C4 at (81.2, 147.4)
- removed the C5 at (81.2, 155.0)
- removed the C6 at (76.0, 168.0)
- removed the C8 at (81.2, 167.5)
- removed the C9 at (85.6, 147.4)
- removed the D1 at (56.7, 142.9)
- removed the D2 at (81.9, 170.5)
- removed the D3 at (81.9, 173.9)
- removed the D4 at (81.9, 177.2)
- removed the D5 at (88.8, 171.0)
- removed the J1 at (139.2, 45.2)
- removed the L1 at (87.8, 176.1)
- removed Q3, Q4: FDS6690A, Package_SO:SOIC-8_3.9x4.9mm_P1.27mm
- removed Q5: AO4407A, footprintf:SOIC127P600X175-8N
- removed the R11 at (89.9, 167.5)
- removed the R13 at (85.6, 152.5)
- removed the R14 at (85.6, 149.9)
- removed the R15 at (94.3, 152.5)
- removed the R16 at (85.6, 162.5)
- removed the R17 at (94.3, 155.0)
- removed the R18 at (94.3, 157.5)
- removed the R19 at (89.9, 160.0)
- removed the R2 at (85.6, 157.5)
- removed the R20 at (94.3, 147.4)
- removed the R21 at (94.3, 149.9)
- removed the R22 at (85.6, 160.0)
- removed the R23 at (85.6, 167.5)
- removed the R24 at (89.9, 147.4)
- removed the R25 at (89.9, 149.9)
- removed the R4 at (85.6, 155.0)
- removed the R5 at (85.6, 165.0)
- removed the R6 at (89.9, 152.5)
- removed the R7 at (89.9, 162.5)
- removed the R8 at (89.9, 155.0)
- removed the R9 at (89.9, 165.0)
- removed the U3 at (96.3, 171.9)
- C7: value 0.1uF -> 100uF
- R10: value 100k -> 470k
- moved Q1 175.5 mm to (224.8, 99.0)
- moved Q2 175.5 mm to (224.8, 105.5)
- moved C7 159.2 mm to (231.5, 97.2)
- moved R10 152.5 mm to (231.3, 100.2)
- renumbered C2 to C1, C23 to C10, C24 to C11, C25 to C12, C26 to C13, C27 to C14, C28 to C15, C29 to C16, C30 to C17, C31 to C18, C32 to C19, C3 to C2, C33 to C20, C34 to C21, C35 to C22, C36 to C23, C37 to C24, C38 to C25, C39 to C26, C40 to C27, C41 to C28, C42 to C29, C104 to C3, C43 to C30, C44 to C31, C45 to C32, C46 to C33, C47 to C34, C48 to C35, C49 to C36, C50 to C37, C51 to C38, C52 to C39, C105 to C4, C53 to C40, C54 to C41, C55 to C42, C56 to C43, C57 to C44, C58 to C45, C59 to C46, C60 to C47, C61 to C48, C62 to C49, C103 to C5, C63 to C50, C64 to C51, C65 to C52, C66 to C53, C67 to C54, C68 to C55, C69 to C56, C70 to C57, C71 to C58, C72 to C59, C106 to C6, C73 to C60, C74 to C61, C75 to C62, C76 to C63, C77 to C64, C78 to C65, C79 to C66, C80 to C67, C81 to C68, C82 to C69, C83 to C70, C84 to C71, C85 to C72, C86 to C73, C87 to C74, C88 to C75, C89 to C76, C90 to C77, C91 to C78, C92 to C79, C21 to C8, C93 to C80, C94 to C81, C95 to C82, C96 to C83, C97 to C84, C98 to C85, C99 to C86, C100 to C87, C101 to C88, C102 to C89, C22 to C9, D16 to D1, D17 to D2, D18 to D3, D21 to D4, D19 to D5, IC3 to IC1, IC1 to IC2, IC2 to IC3, J2 to J1, J12 to J2, L4 to L1, R26 to R11, R27 to R12, R28 to R13, R29 to R14, R30 to R15, R31 to R16, R32 to R17, R33 to R18, R34 to R19, R3 to R2, R35 to R20, R36 to R21, R37 to R22, R38 to R23, R39 to R24, R40 to R25, R41 to R26, R42 to R27, R43 to R28, R44 to R29, R53 to R3, R45 to R30, R46 to R31, R47 to R32, R48 to R33, R49 to R34, R50 to R35, R51 to R36, R52 to R37, R54 to R4, R55 to R5, R56 to R6, R57 to R7, R12 to R8, R58 to R9, U20 to U3
Connections:
- C3 pad 1: Net-(D17-A) -> /so_do_khoi/RTU_SENSOR_DATA/BQ24610_POWER_CHARGE/V_ADAPTER
- C7 pad 1: Net-(U3-ACP) -> /so_do_khoi/RTU_SENSOR_DATA/BQ24610_POWER_CHARGE/VSYSTEM
- C7 pad 2: /so_do_khoi/RTU_SENSOR_DATA/BQ24610_POWER_CHARGE/VSYSTEM -> GND
- D2 pad 2: Net-(D17-A) -> /so_do_khoi/RTU_SENSOR_DATA/BQ24610_POWER_CHARGE/V_ADAPTER
- D3 pad 2: Net-(D17-A) -> /so_do_khoi/RTU_SENSOR_DATA/BQ24610_POWER_CHARGE/V_ADAPTER
- IC1 pad 1: Net-(D17-A) -> /so_do_khoi/RTU_SENSOR_DATA/BQ24610_POWER_CHARGE/V_ADAPTER
- Q1 pad 1: Net-(C4-Pad1) -> /so_do_khoi/RTU_SENSOR_DATA/BQ24610_POWER_CHARGE/VSYSTEM
- Q1 pad 2: Net-(C4-Pad1) -> /so_do_khoi/RTU_SENSOR_DATA/BQ24610_POWER_CHARGE/VSYSTEM
- Q1 pad 3: Net-(C4-Pad1) -> /so_do_khoi/RTU_SENSOR_DATA/BQ24610_POWER_CHARGE/VSYSTEM
- Q1 pad 4: Net-(C4-Pad2) -> Net-(U3-GATE)
- Q1 pad 5: VCC -> /so_do_khoi/RTU_SENSOR_DATA/BQ24610_POWER_CHARGE/PACK+
- Q1 pad 6: VCC -> /so_do_khoi/RTU_SENSOR_DATA/BQ24610_POWER_CHARGE/PACK+
- Q1 pad 7: VCC -> /so_do_khoi/RTU_SENSOR_DATA/BQ24610_POWER_CHARGE/PACK+
- Q1 pad 8: VCC -> /so_do_khoi/RTU_SENSOR_DATA/BQ24610_POWER_CHARGE/PACK+
- Q2 pad 1: Net-(C4-Pad1) -> /so_do_khoi/RTU_SENSOR_DATA/BQ24610_POWER_CHARGE/VSYSTEM
- Q2 pad 2: Net-(C4-Pad1) -> /so_do_khoi/RTU_SENSOR_DATA/BQ24610_POWER_CHARGE/VSYSTEM
- Q2 pad 3: Net-(C4-Pad1) -> /so_do_khoi/RTU_SENSOR_DATA/BQ24610_POWER_CHARGE/VSYSTEM
- Q2 pad 4: Net-(C4-Pad2) -> Net-(U3-STAT)
- Q2 pad 5: Net-(U3-ACP) -> /so_do_khoi/RTU_SENSOR_DATA/BQ24610_POWER_CHARGE/V_ADAPTER
- Q2 pad 6: Net-(U3-ACP) -> /so_do_khoi/RTU_SENSOR_DATA/BQ24610_POWER_CHARGE/V_ADAPTER
- Q2 pad 7: Net-(U3-ACP) -> /so_do_khoi/RTU_SENSOR_DATA/BQ24610_POWER_CHARGE/V_ADAPTER
- Q2 pad 8: Net-(U3-ACP) -> /so_do_khoi/RTU_SENSOR_DATA/BQ24610_POWER_CHARGE/V_ADAPTER
- R10 pad 1: /so_do_khoi/RTU_SENSOR_DATA/BQ24610_POWER_CHARGE/VREF -> /so_do_khoi/RTU_SENSOR_DATA/BQ24610_POWER_CHARGE/VSYSTEM
- R10 pad 2: Net-(U3-ISET1) -> Net-(U3-STAT)
- R3 pad 2: Net-(D17-A) -> /so_do_khoi/RTU_SENSOR_DATA/BQ24610_POWER_CHARGE/V_ADAPTER
- R4 pad 1: Net-(D17-A) -> /so_do_khoi/RTU_SENSOR_DATA/BQ24610_POWER_CHARGE/V_ADAPTER
- U3 pad 1: unconnected-(U20-VIN-Pad1) -> /so_do_khoi/RTU_SENSOR_DATA/BQ24610_POWER_CHARGE/PACK+
- U3 pad 2: unconnected-(U20-GND-Pad2) -> GND
- U3 pad 3: unconnected-(U20-CTL-Pad3) -> GND
- U3 pad 4: unconnected-(U20-STAT-Pad4) -> Net-(U3-STAT)
- U3 pad 5: unconnected-(U20-GATE-Pad5) -> Net-(U3-GATE)
- U3 pad 6: unconnected-(U20-SENSE-Pad6) -> /so_do_khoi/RTU_SENSOR_DATA/BQ24610_POWER_CHARGE/VSYSTEM
Routing:
- net (no net): vias 1 -> 0
